Commit message: main launch file added together with lidar link in urdf

File: description/robot.urdf.xacro (robot description, xacro)
@@ -1,23 +1,46 @@
-<?xml version="1.0"?>
 <robot xmlns:xacro="http://www.ros.org/wiki/xacro" name="robot">
     <!-- BASE LINK -->
-    <link name="base_link">
-    </link>
+    <link name="base_link"/>
     <!-- Joint connecting base_link to mpu_link -->
     <joint name="base_to_mpu" type="fixed">
         <parent link="base_link"/>
         <child link="mpu_link"/>
-        <origin xyz="0 0 1" rpy="0 0 0"/>
+        <origin xyz="0 0 0.06" rpy="0 0 0"/>
     </joint>
     <!-- MPU -->
     <link name="mpu_link">
         <visual>
-        <!-- Visual representation of the MPU -->
+            <!-- Visual representation of the MPU -->
         </visual>
         <collision>
-        <!-- Collision model of the MPU -->
+            <!-- Collision model of the MPU -->
         </collision>
         <inertial>
-        <!-- Inertial properties of the MPU -->
+            <!-- Inertial properties of the MPU -->
+            <mass value="1.0"/>
+            <origin xyz="0 0 0" rpy="0 0 0"/>
+            <inertia ixx="0.1" ixy="0.0" ixz="0.0" iyy="0.1" iyz="0.0" izz="0.1"/>
+        </inertial>
+        <origin xyz="0 0 0" rpy="0 0 0"/>
+    </link>
+    <!-- Joint connecting base_link to lidar_link -->
+    <joint name="base_to_lidar" type="fixed">
+        <parent link="base_link"/>
+        <child link="lidar_link"/>
+        <origin xyz="0 0 0.11" rpy="0 0 0"/>
+    </joint>
+    <!-- LIDAR -->
+    <link name="lidar_link">
+        <visual>
+            <!-- Visual representation of the Lidar -->
+        </visual>
+        <collision>
+            <!-- Collision model of the Lidar -->
+        </collision>
+        <inertial>
+            <!-- Inertial properties of the Lidar -->
+            <mass value="1.0"/>
+            <origin xyz="0 0 0" rpy="0 0 0"/>
+            <inertia ixx="0.1" ixy="0.0" ixz="0.0" iyy="0.1" iyz="0.0" izz="0.1"/>
         </inertial>
         <origin xyz="0 0 0" rpy="0 0 0"/>

Commit message: tf between lidar and world works

File: description/robot.urdf.xacro (robot description, xacro)
@@ -28,5 +28,5 @@
         <parent link="base_link"/>
         <child link="lidar_link"/>
-        <origin xyz="0 0 0.11" rpy="0 0 0"/>
+        <origin xyz="0 0 2.11" rpy="0 0 0"/>
     </joint>
     <!-- LIDAR -->

Commit message: tfs are working. Distortion is compensated, but there is a slight delay

File: description/robot.urdf.xacro (robot description, xacro)
@@ -28,5 +28,5 @@
         <parent link="base_link"/>
         <child link="lidar_link"/>
-        <origin xyz="0 0 2.11" rpy="0 0 0"/>
+        <origin xyz="0 0 0.11" rpy="0 0 0"/>
     </joint>
     <!-- LIDAR -->
